File: 16 ch sample-and-hold card - single-sided - w logo - inc vca - panelized - ordered 180802.brd (EAGLE design)
At the start: 99.8 x 99.6 mm, 361 parts, among them IC1 MAX306CWI, IC10 MAX306CWI, IC11 TL074D, IC12 TL074D, IC13 TL074D, IC14 TL074D, IC15 MAX306CWI, IC16 TL074D, IC17 TL074D, IC18 TL074D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

Commit message: Added logo
Parts:
- R137, R139: value 27k -> 12k
- R141, R142: value 88k2 -> 8k2
Changed lines of the file:
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@@
 <attribute name="VALUE" x="75.184" y="76.073" size="1.27" layer="27" ratio="10"/>
 </element>
-<element name="R137" library="resistor" package="R0805" value="27k" x="83.3755" y="73.2155" smashed="yes" rot="MR90">
+<element name="R137" library="resistor" package="R0805" value="12k" x="83.3755" y="73.2155" smashed="yes" rot="MR90">
 <attribute name="VALUE" x="81.0895" y="72.4535" size="1.27" layer="28" rot="MR90"/>
 </element>
@@
 <attribute name="VALUE" x="83.1215" y="73.9775" size="1.27" layer="28" rot="MR270"/>
 </element>
-<element name="R139" library="resistor" package="R0805" value="27k" x="83.3755" y="80.2005" smashed="yes" rot="MR270">
+<element name="R139" library="resistor" package="R0805" value="12k" x="83.3755" y="80.2005" smashed="yes" rot="MR270">
 <attribute name="VALUE" x="85.6615" y="80.9625" size="1.27" layer="28" rot="MR270"/>
 </element>
@@
 <attribute name="VALUE" x="78.5495" y="79.4385" size="1.27" layer="28" rot="MR90"/>
 </element>
-<element name="R141" library="resistor" package="R0805" value="88k2" x="78.2955" y="73.533" smashed="yes" rot="MR90">
+<element name="R141" library="resistor" package="R0805" value="8k2" x="78.2955" y="73.533" smashed="yes" rot="MR90">
 <attribute name="VALUE" x="76.0095" y="72.771" size="1.27" layer="28" rot="MR90"/>
 </element>
-<element name="R142" library="resistor" package="R0805" value="88k2" x="78.2955" y="79.883" smashed="yes" rot="MR270">
+<element name="R142" library="resistor" package="R0805" value="8k2" x="78.2955" y="79.883" smashed="yes" rot="MR270">
 <attribute name="VALUE" x="80.5815" y="80.645" size="1.27" layer="28" rot="MR270"/>
 </element>
