File: Simplified 4 ch sample-and-hold without mux v2.0.sch (EAGLE design)
At the start: 8 parts, among them IC5 TL074JT

Commit message: Fixed error in silk screen
Parts:
- IC5: value TL074JT -> TL084CPWR
Changed lines of the file:
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@@
 <?xml version="1.0" encoding="utf-8"?>
 <!DOCTYPE eagle SYSTEM "eagle.dtd">
-<eagle version="9.5.2">
+<eagle version="9.6.2">
 <drawing>
 <settings>
@@
 <part name="P+1" library="supply1" deviceset="+15V" device=""/>
 <part name="P-1" library="supply1" deviceset="-15V" device=""/>
-<part name="IC5" library="joakim" deviceset="TL074J" device="T"/>
+<part name="IC5" library="joakim" deviceset="TL074J" device="T" value="TL084CPWR"/>
 <part name="C29" library="rcl" library_urn="urn:adsk.eagle:library:334" deviceset="C-EU" device="C0805" package3d_urn="urn:adsk.eagle:package:23617/2" value="10nF"/>
 <part name="C28" library="rcl" library_urn="urn:adsk.eagle:library:334" deviceset="C-EU" device="C0805" package3d_urn="urn:adsk.eagle:package:23617/2" value="10nF"/>
