File: 16 ch sample-and-hold card v4_1-dual.brd (EAGLE design)
At the start: 76.8 x 24.8 mm, 36 parts, among them IC1 TL074D, IC2 TL074D, IC3 TL074D, IC4 TL074D, IC5 78L05F, IC7 4051D, IC8 4051D

Commit message: moving
Parts:
- added C14, C15, C16, C17, C19, C20, C21, C32, C34, C35, C36, C37, C39, C41, C42, C43: 10nF, rcl:C0805
- added C18, C33, C38, C44, C45, C46, C47: 0.1uF, resistor:C0603
- added C48: 0.33uF, resistor:C0603
- added IC10, IC11, IC6, IC9: TL074D, linear:SO14
- added IC12, IC13: 4051D, 40xx:SO16
- added IC14: 78L05F, linear:SOT89
- added SJ3, SJ4: (no value), jumper:SJ
- added SV1: (no value), joakim:MA20-1
- added SV4: (no value), joakim:MA08-2J
- added U$2: (no value), joakim:XONIK_LOGO_50
Connections:
- new net +15V1: C18.1, C33.1, C38.1, C44.1, C48.2, IC10.4, IC11.4, IC14.3, IC6.4, IC9.4, SV1.18, SV4.2
- new net +5V1: C45.2, C46.2, C47.2, IC12.16, IC13.16, IC14.1
- new net -15V1: C18.2, C33.2, C38.2, C44.2, IC10.11, IC11.11, IC6.11, IC9.11, SV1.19, SV4.1
- new net A3: IC12.11, IC13.11, SV4.8
- new net A4: IC12.10, IC13.10, SV4.7
- new net A5: IC12.9, IC13.9, SV4.10
- new net AGND1: C14.1, C15.1, C16.1, C17.1, C19.1, C20.1, C21.1, C32.1, C34.1, C35.1, C36.1, C37.1, C39.1, C41.1, C42.1, C43.1, SJ3.2, SV1.17, SV4.16
- new net DAC2: IC12.3, SV4.15
- new net DAC3: IC13.3, SV4.13
- new net DGND1: SJ4.1, SV4.5, SV4.6
- new net EN2: IC13.6, SV4.9
- new net EN3: IC12.6, SV4.12
- new net IN_16: C17.2, IC13.13, IC6.12
- new net IN_17: C16.2, IC13.14, IC6.10
- new net IN_18: C15.2, IC13.15, IC6.5
- new net IN_19: C14.2, IC13.12, IC6.3
- new net IN_20: C32.2, IC13.1, IC9.12
- new net IN_21: C21.2, IC13.5, IC9.10
- new net IN_22: C20.2, IC13.2, IC9.5
- new net IN_23: C19.2, IC13.4, IC9.3
- new net IN_24: C34.2, IC10.3, IC12.12
- new net IN_25: C35.2, IC10.5, IC12.15
- new net IN_26: C36.2, IC10.10, IC12.14
- new net IN_27: C37.2, IC10.12, IC12.13
- new net IN_28: C39.2, IC11.3, IC12.4
- new net IN_29: C41.2, IC11.5, IC12.2
- new net IN_30: C42.2, IC11.10, IC12.5
- new net IN_31: C43.2, IC11.12, IC12.1
- new net N$1: C45.1, C46.1, C47.1, C48.1, IC12.7, IC12.8, IC13.7, IC13.8, IC14.2, IC14.2@1, SJ3.1, SJ4.2
- new net OUT_16: IC6.13, IC6.14, SV1.1
- new net OUT_17: IC6.6, IC6.7, SV1.3
- new net OUT_18: IC6.1, IC6.2, SV1.4
- new net OUT_19: IC6.8, IC6.9, SV1.2
- new net OUT_20: IC9.1, IC9.2, SV1.8
- new net OUT_21: IC9.6, IC9.7, SV1.7
- new net OUT_22: IC9.8, IC9.9, SV1.6
- new net OUT_23: IC9.13, IC9.14, SV1.5
- new net OUT_24: IC10.1, IC10.2, SV1.12
- new net OUT_25: IC10.6, IC10.7, SV1.11
- new net OUT_26: IC10.8, IC10.9, SV1.10
- new net OUT_27: IC10.13, IC10.14, SV1.9
- new net OUT_28: IC11.6, IC11.7, SV1.15
- new net OUT_29: IC11.8, IC11.9, SV1.14
- new net OUT_30: IC11.13, IC11.14, SV1.13
- new net OUT_31: IC11.1, IC11.2, SV1.16
Routing:
- net +15V1: track 0.00 -> 121.0 mm, vias 0 -> 2
- net -15V1: track 0.00 -> 119.6 mm, vias 0 -> 7
- net AGND1: track 0.00 -> 93.9 mm, vias 0 -> 1
- net IN_16: track 0.00 -> 73.1 mm, vias 0 -> 2
- net IN_17: track 0.00 -> 72.9 mm, vias 0 -> 2
- net IN_18: track 0.00 -> 70.6 mm, vias 0 -> 2
- net IN_21: track 0.00 -> 69.9 mm, vias 0 -> 2
- net IN_20: track 0.00 -> 67.4 mm, vias 0 -> 2
- net IN_19: track 0.00 -> 65.6 mm, vias 0 -> 2
- net IN_22: track 0.00 -> 64.7 mm, vias 0 -> 2
- net IN_23: track 0.00 -> 60.5 mm, vias 0 -> 2
- net +5V1: track 0.00 -> 52.0 mm, vias 0 -> 3
- net N$1: track 0.00 -> 50.3 mm, vias 0 -> 5
- net IN_27: track 0.00 -> 34.1 mm, vias 0 -> 2
- net IN_26: track 0.00 -> 33.4 mm, vias 0 -> 2
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- added copper zone on layer 16, net DGND1
Other:
- board size 76.8 x 24.8 mm -> 76.8 x 51.8 mm
