File: 56 ch sample-and-hold card v1.0.sch (EAGLE design)
At the start: 143 parts, among them IC1 74HCT4051D, IC10 TL074JT, IC11 74HCT4051D, IC12 TL074JT, IC13 TL074JT, IC14 74HCT4051D, IC15 TL074JT, IC16 TL074JT, IC17 74HCT4051D, IC18 TL074JT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

Commit message: v1.0 ready for production
Parts:
- C2: value 150nF -> 100nF
- IC2: value DAC8586F -> DAC8565F; device joakim:DAC8586F -> joakim:DAC8565F
- U$2, U$3, U$4: value FEMALE -> MA15-2J-FEMALE
- X10: value FEMALE -> MA07-2J-FEMALE
- X6: value FEMALE -> MA08-2J-FEMALE
Changed lines of the file:
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@@
 <part name="C119" library="joakim" deviceset="C-EU-J" device="0402" value="1uF"/>
 <part name="AGND101" library="supply1" deviceset="AGND" device=""/>
-<part name="IC2" library="joakim" deviceset="DAC8586" device="F" value="DAC8586F"/>
+<part name="IC2" library="joakim" deviceset="DAC8565" device="F" value="DAC8565F"/>
 <part name="AGND1" library="supply1" deviceset="AGND" device=""/>
 <part name="AGND6" library="supply1" deviceset="AGND" device=""/>
-<part name="C2" library="resistor" deviceset="C-EU" device="C0603" value="150nF"/>
+<part name="C2" library="resistor" deviceset="C-EU" device="C0603" value="100nF"/>
 <part name="AGND9" library="supply1" deviceset="AGND" device=""/>
 <part name="AGND11" library="supply1" deviceset="AGND" device=""/>
@@
 <part name="R11" library="rcl" library_urn="urn:adsk.eagle:library:334" deviceset="R-EU_" device="R0603" package3d_urn="urn:adsk.eagle:package:23555/3" value="220R"/>
 <part name="R12" library="rcl" library_urn="urn:adsk.eagle:library:334" deviceset="R-EU_" device="R0603" package3d_urn="urn:adsk.eagle:package:23555/3" value="220R"/>
-<part name="X6" library="joakim" deviceset="MA08-2J" device="" value="FEMALE"/>
-<part name="X10" library="joakim" deviceset="MA07-2J" device="" value="FEMALE"/>
-<part name="U$2" library="joakim" deviceset="MA15-2J" device="" value="FEMALE"/>
-<part name="U$3" library="joakim" deviceset="MA15-2J" device="" value="FEMALE"/>
-<part name="U$4" library="joakim" deviceset="MA15-2J" device="" value="FEMALE"/>
+<part name="X6" library="joakim" deviceset="MA08-2J" device="" value="MA08-2J-FEMALE"/>
+<part name="X10" library="joakim" deviceset="MA07-2J" device="" value="MA07-2J-FEMALE"/>
+<part name="U$2" library="joakim" deviceset="MA15-2J" device="" value="MA15-2J-FEMALE"/>
+<part name="U$3" library="joakim" deviceset="MA15-2J" device="" value="MA15-2J-FEMALE"/>
+<part name="U$4" library="joakim" deviceset="MA15-2J" device="" value="MA15-2J-FEMALE"/>
 <part name="C5" library="joakim" deviceset="C-EU-J" device="0402" value="1uF"/>
 <part name="P+1" library="supply2" library_urn="urn:adsk.eagle:library:372" deviceset="+12V" device=""/>

Commit message: Added comment
Other:
- note added: "2 x gain, changes 2.5V at DAC to 5V at CV buffers"
Changed lines of the file:
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@@
 <text x="-48.26" y="43.18" size="1.778" layer="91">TODO: Pulldown på LDAC</text>
 <text x="175.26" y="88.9" size="1.778" layer="91">TODO: FIX NAMING!</text>
+<text x="132.08" y="88.9" size="1.778" layer="97">2 x gain, changes 2.5V at
+DAC to 5V at CV buffers</text>
 </plain>
 <instances>
