File: level-shifter-v1.0.brd (EAGLE design)
At the start: 15.2 x 10.2 mm, 8 parts, among them IC1 SN74LVC2T45, IC2 SN74LVC2T45, X1 MA06-1JC, X2 MA06-1JC

Commit message: Updated footprint
Parts:
- X1, X2: value MA06-1JC -> MA06-1JN; device joakim:MA06-1J -> joakim:MA06N-1J
Routing:
- net GND: track 4.17 -> 4.98 mm
- net A4: track 5.74 -> 5.09 mm
- net A2: track 7.24 -> 6.59 mm
- net B1: track 6.00 -> 5.45 mm
- net A1: track 5.43 -> 4.87 mm
Other:
- board text added: "4 x Logic level shifter"
- board text added: "A1"
- board text added: "A2"
- board text added: "A3"
- board text added: "A4"
- board text added: "B1"
- board text added: "B2"
- board text added: "B3"
- board text added: "B4"
- board text added: "D:VA=A B, 0=B A"
- board text added: "Dir"
- board text added: "Gd"
- board text added: "VA"
- board text added: "VB"
- board text added: "v1.0"
