File: level-shifter-v1.0.sch (EAGLE design)
At the start: 8 parts, among them IC1 SN74LVC2T45, IC2 SN74LVC2T45, X1 MA06-1JC, X2 MA06-1JC

Commit message: Updated footprint
Parts:
- X1, X2: value MA06-1JC -> MA06-1JN; device joakim:MA06-1JC -> joakim:MA06-1JN
Changed lines of the file:
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@@
 <part name="P+2" library="supply1" library_urn="urn:adsk.eagle:library:371" deviceset="+5V" device=""/>
 <part name="GND6" library="supply1" library_urn="urn:adsk.eagle:library:371" deviceset="GND" device=""/>
-<part name="X1" library="joakim" deviceset="MA06-1J" device="C"/>
-<part name="X2" library="joakim" deviceset="MA06-1J" device="C"/>
+<part name="X1" library="joakim" deviceset="MA06-1J" device="N" value="MA06-1JN"/>
+<part name="X2" library="joakim" deviceset="MA06-1J" device="N" value="MA06-1JN"/>
 <part name="+3V3" library="supply1" library_urn="urn:adsk.eagle:library:371" deviceset="+3V3" device=""/>
 <part name="P+3" library="supply1" library_urn="urn:adsk.eagle:library:371" deviceset="+5V" device=""/>
